File: rj11-breakout.sch (EAGLE design)
At the start: 2 parts, among them J1 22-27-2061-06, X1 XRJK-S-01-6-6-0-2G2-NO

Commit message: changed to correct RJ11 part
Parts:
- removed X1: XRJK-S-01-6-6-0-2G2-NO, con-xmultiple:XRJK-S-01-6-6-0-2G2-NO
- added J2: RJ11-6L-B, con-tycoelectronics:RJ11-6L-B
Connections:
- net N$1: now also J1-1.S, J2.6; no longer J1-6.S, X1.1
- net N$2: now also J1-2.S, J2.5; no longer J1-5.S, X1.2
- net N$3: now also J1-3.S, J2.4; no longer J1-4.S, X1.3
- net N$4: now also J1-4.S, J2.3; no longer J1-3.S, X1.4
- net N$5: now also J1-5.S, J2.2; no longer J1-2.S, X1.5
- net N$6: now also J1-6.S, J2.1; no longer J1-1.S, X1.6
Changed lines of the file:
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@@
 </classes>
 <parts>
-<part name="X1" library="con-xmultiple" deviceset="XRJK*6" device="-0-2G2-NO" technology="-S-01-6-"/>
 <part name="J1" library="con-molex" deviceset="22-?-06" device="27-2061"/>
+<part name="J2" library="con-tycoelectronics" deviceset="RJ11" device="" technology="-6L-B"/>
 </parts>
 <sheets>
@@
 </plain>
 <instances>
-<instance part="X1" gate="G$1" x="53.34" y="48.26"/>
 <instance part="J1" gate="-1" x="43.18" y="43.18" rot="R180"/>
 <instance part="J1" gate="-2" x="43.18" y="45.72" rot="R180"/>
@@
 <instance part="J1" gate="-5" x="43.18" y="53.34" rot="R180"/>
 <instance part="J1" gate="-6" x="43.18" y="55.88" rot="R180"/>
+<instance part="J2" gate="G$1" x="50.8" y="50.8"/>
 </instances>
 <busses>
@@
 <net name="N$1" class="0">
 <segment>
-<pinref part="X1" gate="G$1" pin="1"/>
-<pinref part="J1" gate="-6" pin="S"/>
+<pinref part="J1" gate="-1" pin="S"/>
+<pinref part="J2" gate="G$1" pin="6"/>
+<wire x1="48.26" y1="43.18" x2="45.72" y2="43.18" width="0.1524" layer="91"/>
 </segment>
 </net>
 <net name="N$2" class="0">
 <segment>
-<pinref part="X1" gate="G$1" pin="2"/>
-<pinref part="J1" gate="-5" pin="S"/>
+<pinref part="J1" gate="-2" pin="S"/>
+<pinref part="J2" gate="G$1" pin="5"/>
+<wire x1="48.26" y1="45.72" x2="45.72" y2="45.72" width="0.1524" layer="91"/>
 </segment>
 </net>
 <net name="N$3" class="0">
 <segment>
-<pinref part="X1" gate="G$1" pin="3"/>
-<pinref part="J1" gate="-4" pin="S"/>
+<pinref part="J1" gate="-3" pin="S"/>
+<pinref part="J2" gate="G$1" pin="4"/>
+<wire x1="48.26" y1="48.26" x2="45.72" y2="48.26" width="0.1524" layer="91"/>
 </segment>
 </net>
 <net name="N$4" class="0">
 <segment>
-<pinref part="X1" gate="G$1" pin="4"/>
-<pinref part="J1" gate="-3" pin="S"/>
+<pinref part="J1" gate="-4" pin="S"/>
+<pinref part="J2" gate="G$1" pin="3"/>
+<wire x1="48.26" y1="50.8" x2="45.72" y2="50.8" width="0.1524" layer="91"/>
 </segment>
 </net>
 <net name="N$5" class="0">
 <segment>
-<pinref part="X1" gate="G$1" pin="5"/>
-<pinref part="J1" gate="-2" pin="S"/>
+<pinref part="J1" gate="-5" pin="S"/>
+<pinref part="J2" gate="G$1" pin="2"/>
+<wire x1="48.26" y1="53.34" x2="45.72" y2="53.34" width="0.1524" layer="91"/>
 </segment>
 </net>
 <net name="N$6" class="0">
 <segment>
-<pinref part="X1" gate="G$1" pin="6"/>
-<pinref part="J1" gate="-1" pin="S"/>
+<pinref part="J1" gate="-6" pin="S"/>
+<pinref part="J2" gate="G$1" pin="1"/>
+<wire x1="48.26" y1="55.88" x2="45.72" y2="55.88" width="0.1524" layer="91"/>
 </segment>
 </net>
